File: stm_main/stlink.kicad_sch (KiCad schematic)
At the start: 21 parts, among them IC5 STM32F103CBT6, J7 Conn_01x05_Pin, Y2 XVHCELNANF

Commit message: ✨feat:発注8/27
Connections:
- net RENUM: no longer names the net of IC5.38 (PA15)
- net T_RST: no longer names the net of IC5.18 (PB0)
- net T_RX: no longer names the net of IC5.13 (PA3)
- net T_SWO: no longer names the net of IC5.31 (PA10)
- net T_TX: no longer names the net of IC5.12 (PA2)
- no-connect marks 0 -> 24
