File: stm_main/stm_main.kicad_pcb (KiCad board)
At the start: 2 copper layers, 70 x 85 mm, 99 parts, among them IC1 USBLC6-2SC6, IC2 STM32F405RGT6TR, IC3 MCP1703AT-3302E_CB, IC4 MAX3051EKA+T, IC5 STM32F103CBT6, J1 MUSB-5BF01AS, J2 XN2D-1471, J3 XN2D-1471, J4 XN2D-1471, J5 XN2D-1471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

Commit message: ✨feat:発注8/27
Parts:
- added R29: 10, Resistor_SMD:R_0603_1608Metric, F.Cu at (64.0, 33.0)
- added R30: 0, Resistor_SMD:R_0603_1608Metric, F.Cu at (23.6, 83.8)
- J2, J3, J4, J5: value XN2D-1471 -> B04B-XASK-1_LF__SN_; footprint my_pretty:XN2D1471 -> my_pretty:SHDR4W60P0X250_1X4_1250X640X880P
- J6: value XN2D-1671 -> B06B-XASK-1_LF__SN_; footprint my_pretty:XN2D1671 -> my_pretty:SHDR6W80P0X250_1X6_1750X640X880P
- R1, R2, R3: value 330 -> 0
- R10: value 1k -> 510
- R12: value 500 -> 150
- R13: value 330 -> 82
- R5: value 340 -> 330
- moved C5 13.1 mm to (37.6, 83.8), turned to 180 degrees
- moved J6 9.68 mm to (37.1, 89.7)
- moved R3 8.41 mm to (27.0, 83.8), turned to 180 degrees
- moved R1 6.39 mm to (34.2, 83.8), turned to 180 degrees
- moved J2 4.60 mm to (32.0, 58.4)
- moved J3 4.60 mm to (32.0, 67.6)
- moved J4 4.60 mm to (32.0, 35.1)
- moved J5 4.60 mm to (32.0, 44.2)
- moved R2 1.91 mm to (30.5, 83.8), turned to 180 degrees
Connections:
- IC2 pad 54: /PD2 -> unconnected-(IC2-PD2-Pad54)
- IC5 pad 12: /stlink/T_TX -> unconnected-(IC5-PA2-Pad12)
- IC5 pad 13: /stlink/T_RX -> unconnected-(IC5-PA3-Pad13)
- IC5 pad 18: /stlink/T_RST -> unconnected-(IC5-PB0-Pad18)
- IC5 pad 31: /stlink/T_SWO -> unconnected-(IC5-PA10-Pad31)
- IC5 pad 38: /stlink/RENUM -> unconnected-(IC5-PA15-Pad38)
- J6 pad 6: /PC0 -> Net-(J6-Pad6)
- R5 pad 2: GND -> Net-(R29-Pad1)
Routing:
- net /USART0_RX: track 31.5 -> 42.8 mm
- net /USART1_RX: track 38.3 -> 49.1 mm
- net /CAN0_L: track 19.7 -> 29.0 mm
- net +5V: track 146.0 -> 138.0 mm
- net Net-(J6-Pad6): track 0.00 -> 6.59 mm
- net /USART0_TX: track 35.6 -> 40.6 mm
- net /USART1_TX: track 40.0 -> 44.4 mm
- net /CAN0_H: track 29.4 -> 33.7 mm
- net Net-(R29-Pad1): track 0.00 -> 3.54 mm
- net GND: track 43.2 -> 45.2 mm, vias 258 -> 270
- net Net-(J6-Pad5): track 7.64 -> 6.23 mm
- net Net-(J6-Pad2): track 7.60 -> 6.34 mm
- net Net-(J6-Pad3): track 7.83 -> 6.83 mm
