File: stm_main/stm_main.kicad_sch (KiCad schematic)
At the start: 73 parts, among them IC1 USBLC6-2SC6, IC2 STM32F405RGT6TR, IC3 MCP1703AT-3302E_CB, IC4 MAX3051EKA+T, J1 MUSB-5BF01AS, J2 XN2D-1471, J3 XN2D-1471, J4 XN2D-1471, J5 XN2D-1471, J6 XN2D-1671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

Commit message: ✨feat:発注8/27
Parts:
- removed J2, J3, J4, J5: XN2D-1471, my_pretty:XN2D1471, symbol my_library:XN2D-1471
- removed J6: XN2D-1671, my_pretty:XN2D1671, symbol my_library:XN2D-1671
- added J2, J3, J4, J5: B04B-XASK-1_LF__SN_, my_pretty:SHDR4W60P0X250_1X4_1250X640X880P, symbol my_library:B04B-XASK-1_LF__SN_
- added J6: B06B-XASK-1_LF__SN_, my_pretty:SHDR6W80P0X250_1X6_1750X640X880P, symbol my_library:B06B-XASK-1_LF__SN_
- added R29: 10, Resistor_SMD:R_0603_1608Metric, symbol Device:R
- added R30: 0, Resistor_SMD:R_0603_1608Metric, symbol Device:R
- R1, R2, R3: value 330 -> 0
- R10: value 1k -> 510
- R12: value 500 -> 150
- R13: value 330 -> 82
- R5: value 340 -> 330
Connections:
- net +5V: now also J2.2, J3.2, J6.1
- net CAN0_H: now also J4.3, J5.3
- net CAN0_L: now also J4.4, J5.4
- net GND: now also J2.1, J3.1, J4.1, J5.1, J6.4, R29.2; no longer R5.2
- net PC0: now also R30.1
- net USART0_RX: now also J2.4
- net USART0_TX: now also J2.3
- net USART1_RX: now also J3.4
- net USART1_TX: now also J3.3
- net at C1.2, C2.1, D1.2 (A): now also J4.2, J5.2
- net at R1.2: now also J6.2
- net at R2.2: now also J6.3
- net at R3.2: now also J6.5
- net PD2: no longer names the net of IC2.54 (PD2)
- new net: J6.6, R30.2
- new net: R29.1, R5.2
- no-connect marks 4 -> 49
Other:
- moved on the sheet: R11, R4, R5, SW1, SW2

Commit message: 🍰chore:sch
Parts:
- R10: value 510 -> 2k
- R12: value 150 -> 560
- R13: value 82 -> 270
Changed lines of the file:
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@@
   (junction (at 137.16 63.5) (diameter 0) (color 0 0 0 0)
   )
-  (junction (at 320.04 128.27) (diameter 0) (color 0 0 0 0)
-  )
   (junction (at 138.43 229.87) (diameter 0) (color 0 0 0 0)
   )
@@
     (stroke (width 0) (type default))
   )
+  (wire (pts (xy 320.04 127) (xy 320.04 128.27))
+    (stroke (width 0) (type default))
+  )
   (wire (pts (xy 171.45 243.84) (xy 171.45 252.73))
     (stroke (width 0) (type default))
@@
     (stroke (width 0) (type default))
   )
-  (wire (pts (xy 320.04 128.27) (xy 320.04 128.905))
-    (stroke (width 0) (type default))
-  )
   (wire (pts (xy 190.5 273.05) (xy 190.5 275.59))
     (stroke (width 0) (type default))
@@
     (stroke (width 0) (type default))
   )
-  (wire (pts (xy 320.04 127) (xy 320.04 128.27))
-    (stroke (width 0) (type default))
-  )
   (wire (pts (xy 40.64 144.78) (xy 40.64 143.51))
     (stroke (width 0) (type default))
@@
       (effects (font (size 1.27 1.27)) (justify left))
     )
-    (property "Value" "510" (at 318.77 231.14 0)
+    (property "Value" "2k" (at 318.77 231.14 0)
       (effects (font (size 1.27 1.27)) (justify left))
     )
@@
       (effects (font (size 1.27 1.27)) (justify left))
     )
-    (property "Value" "150" (at 328.93 231.14 0)
+    (property "Value" "560" (at 328.93 231.14 0)
       (effects (font (size 1.27 1.27)) (justify left))
     )
@@
       (effects (font (size 1.27 1.27)) (justify left))
     )
-    (property "Value" "82" (at 339.09 231.14 0)
+    (property "Value" "270" (at 339.09 231.14 0)
       (effects (font (size 1.27 1.27)) (justify left))
     )
