File: raspberrypi_hat/raspberrypi_hat.kicad_pcb (KiCad board)
At the start: 2 copper layers, 36.2 x 52.7 mm, 19 parts, among them IC1 MCP2515-I_P, IC2 MCP2562FD-E_P, J1 Conn_02x20_Odd_Even, Y1 Resonator

Commit message: ✨feat:シルク
Parts:
- moved G*** 46.7 mm to (46.0, 79.0)
Changed lines of the file:
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@@
   )
   (footprint "logo_pretty:rdclab_small" (layer "B.Cu")
-    (at 54.356 33.02 180)
+    (at 45.974 78.994 180)
     (attr board_only exclude_from_pos_files exclude_from_bom)
     (fp_text reference "G***" (at 0 0) (layer "B.SilkS") hide
